Commit message: Changed robot tool offset

File: assets/ur5_tool/ur5_tool.urdf (robot description, URDF)
Before this commit: robot ur5_tool, 13 links, 12 joints
Joints:
- joint tool_jt: origin xyz=0.4 0 0 rpy=3.142 -1.571 0 -> xyz=0.28 0 0 rpy=3.142 -1.571 0

Commit message: Tilted base to move singularity from workspace

File: assets/ur5_tool/ur5_tool.urdf (robot description, URDF)
Before this commit: robot ur5_tool, 13 links, 12 joints
Joints:
- joint world_joint: origin xyz=0 0.0 2.3 rpy=0 3.14 0 -> xyz=0 0.0 2.3 rpy=0.785 3.14 0
